Commit message: edit some files

File: formular_car/car.urdf (robot description, URDF)
Before this commit: robot formular_car, 13 links, 11 joints
Links:
- removed link sus_fl
- removed link sus_fr
- removed link sus_rl
- removed link sus_rr
- added link susp_fl, mass 1e-5
- added link susp_fr, mass 1e-5
- added link susp_rl, mass 1e-5
- added link susp_rr, mass 1e-5
- link body: mass 300.0 -> 600.0
- link steering_fl: mass 0.001 -> 1e-5
- link steering_fr: mass 0.001 -> 1e-5
- link steering_rl: mass 0.001 -> 1e-5
- link steering_rr: mass 0.001 -> 1e-5
Joints:
- removed joint steering_fl_joint
- removed joint steering_fr_joint
- removed joint steering_rl_joint
- removed joint steering_rr_joint
- removed joint sus_fl_joint
- removed joint sus_fr_joint
- removed joint sus_rl_joint
- removed joint wheel_fl_joint
- removed joint wheel_fr_joint
- removed joint wheel_rl_joint
- removed joint wheel_rr_joint
- added joint steer_joint_fl: type revolute, parent susp_fl, child steering_fl, axis 0.0 0.0 1.0, limit lower=-0.524 upper=0.524 effort=80 velocity=100
- added joint steer_joint_fr: type revolute, parent susp_fr, child steering_fr, axis 0.0 0.0 1.0, limit lower=-0.524 upper=0.524 effort=80 velocity=100
- added joint steer_joint_rl: type fixed, parent susp_rl, child steering_rl
- added joint steer_joint_rr: type fixed, parent susp_rr, child steering_rr
- added joint susp_joint_fl: type prismatic, parent body, child susp_fl, origin xyz=-1.0 1.4 0.05 rpy=0.0 0.0 0.0, axis 0.0 0.0 1.0, limit lower=-0.1 upper=0.01 effort=500 velocity=1.0
- added joint susp_joint_fr: type prismatic, parent body, child susp_fr, origin xyz=1.0 1.4 0.05 rpy=0.0 0.0 0.0, axis 0.0 0.0 1.0, limit lower=-0.1 upper=0.01 effort=500 velocity=1.0
- added joint susp_joint_rl: type prismatic, parent body, child susp_rl, origin xyz=-1.05 -1.5 0.08 rpy=0.0 0.0 0.0, axis 0.0 0.0 1.0, limit lower=-0.1 upper=0.01 effort=500 velocity=1.0
- added joint susp_joint_rr: type prismatic, parent body, child susp_rr, origin xyz=1.05 -1.5 0.08 rpy=0.0 0.0 0.0, axis 0.0 0.0 1.0, limit lower=-0.1 upper=0.01 effort=500 velocity=1.0
- added joint wheel_joint_fl: type continuous, parent steering_fl, child wheel_fl, axis 1.0 0.0 0.0
- added joint wheel_joint_fr: type continuous, parent steering_fr, child wheel_fr, axis 1.0 0.0 0.0
- added joint wheel_joint_rl: type continuous, parent steering_rl, child wheel_rl, axis 1.0 0.0 0.0
- added joint wheel_joint_rr: type continuous, parent steering_rr, child wheel_rr, axis 1.0 0.0 0.0

Commit message: add new foler

File: formular_car/car.urdf (robot description, URDF)
Before this commit: robot formular_car, 13 links, 12 joints
Links:
- link body: geometry collision mesh filename=./components/body.stl scale=1.0; visual mesh filename=./components/body.stl scale=1.0
- link wheel_fl: geometry collision mesh filename=./components/wheel_FL.stl scale=1.0; visual mesh filename=./components/wheel_FL.stl scale=1.0
- link wheel_fr: geometry collision mesh filename=./components/wheel_FR.stl scale=1.0; visual mesh filename=./components/wheel_FR.stl scale=1.0
- link wheel_rl: geometry collision mesh filename=./components/wheel_RL.stl scale=1.0; visual mesh filename=./components/wheel_RL.stl scale=1.0
- link wheel_rr: geometry collision mesh filename=./components/wheel_RR.stl scale=1.0; visual mesh filename=./components/wheel_RR.stl scale=1.0

Commit message: edit print

File: formular_car/car.urdf (robot description, URDF)
Before this commit: robot formular_car, 13 links, 12 joints
Joints:
- joint susp_joint_fl: limit lower=-0.1 upper=0.01 effort=500 velocity=1.0 -> lower=-0.1 upper=0.08 effort=500 velocity=1.0
- joint susp_joint_fr: limit lower=-0.1 upper=0.01 effort=500 velocity=1.0 -> lower=-0.1 upper=0.08 effort=500 velocity=1.0
- joint susp_joint_rl: limit lower=-0.1 upper=0.01 effort=500 velocity=1.0 -> lower=-0.1 upper=0.08 effort=500 velocity=1.0
- joint susp_joint_rr: limit lower=-0.1 upper=0.01 effort=500 velocity=1.0 -> lower=-0.1 upper=0.08 effort=500 velocity=1.0

Commit message: Completed car.urdf

File: formular_car/car.urdf (robot description, URDF)
Before this commit: robot formular_car, 13 links, 12 joints
Links:
- removed link susp_fl
- removed link susp_fr
- removed link susp_rl
- removed link susp_rr
Joints:
- removed joint susp_joint_fl
- removed joint susp_joint_fr
- removed joint susp_joint_rl
- removed joint susp_joint_rr
- joint steer_joint_fl: limit lower=-0.524 upper=0.524 effort=80 velocity=100 -> lower=-0.5 upper=0.5 effort=80 velocity=100; origin (none) -> xyz=-1.05 1.4 0.09 rpy=0.0 0.0 0.0; parent susp_fl -> body
- joint steer_joint_fr: limit lower=-0.524 upper=0.524 effort=80 velocity=100 -> lower=-0.5 upper=0.5 effort=80 velocity=100; origin (none) -> xyz=1.05 1.4 0.09 rpy=0.0 0.0 0.0; parent susp_fr -> body
- joint steer_joint_rl: origin (none) -> xyz=-1.05 -1.5 0.12 rpy=0.0 0.0 0.0; parent susp_rl -> body
- joint steer_joint_rr: origin (none) -> xyz=1.05 -1.5 0.12 rpy=0.0 0.0 0.0; parent susp_rr -> body
